File: KiCad/Devkit/Hotswap Pico Hub/DevkitHotswapPicoHub.kicad_pcb (KiCad board)
At the start: 2 copper layers, 124.5 x 109.2 mm, 38 parts, among them J202 OS SWD In, J303 User SWD In, J400 OS UART, J401 OS SWD, J404 User UART, J405 User SWD, J502 Devkit Hotswap Hub Port, SW403 OS Reset Switch, SW406 User Reset Switch, U200 OS Pico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

Commit message: Updated KiCad to V1.1.2
Parts:
- added J502.15: TestPoint, TestPoint:TestPoint_Pad_1.5x1.5mm, F.Cu at (122.4, 19.8)
- added J502.17: TestPoint, TestPoint:TestPoint_Pad_1.5x1.5mm, F.Cu at (122.4, 15.9)
- added J502.19: TestPoint, TestPoint:TestPoint_Pad_1.5x1.5mm, F.Cu at (118.7, 15.9)
- added J502.4: TestPoint, TestPoint:TestPoint_Pad_1.5x1.5mm, F.Cu at (118.7, 19.8)
- added Q507: 2N3904, Package_TO_SOT_THT:TO-92_Inline, F.Cu at (92.7, 55.4)
- added R302: 10k, Resistor_SMD:R_0805_2012Metric, F.Cu at (102.0, 49.5)
- added R505: 10k, Resistor_SMD:R_0805_2012Metric, F.Cu at (97.8, 60.0)
- added R506: 10k, Resistor_SMD:R_0805_2012Metric, F.Cu at (94.0, 50.4)
- D409: value User Enable Bus 2 -> User Request Bus 1
- moved R301 45.4 mm to (121.9, 52.7), turned to 0 degrees
- moved R420 2.54 mm to (83.2, 36.2)
- moved R421 2.54 mm to (89.5, 36.2)
- moved R416 2.54 mm to (47.6, 36.2)
- moved R417 2.54 mm to (54.0, 36.2)
- moved R503 2.26 mm to (82.9, 57.8)
Connections:
- D407 pad 1: Net-(D407-K) -> User Enable Bus 1
- D407 pad 2: OS Enable Bus 1 -> Net-(D407-A)
- D408 pad 1: OS Enable Bus 1 -> Net-(D408-K)
- D408 pad 2: Net-(D408-A) -> User Enable Bus 1
- D410 pad 1: ~{User RUN} -> Net-(D410-K)
- D410 pad 2: Net-(D410-A) -> User RUN
- D411 pad 1: Net-(D411-K) -> User Enable Bus 2
- D411 pad 2: OS Enable Bus 2 -> Net-(D411-A)
- D412 pad 1: OS Enable Bus 2 -> Net-(D412-K)
- D412 pad 2: Net-(D412-A) -> User Enable Bus 2
- J502 pad 1: GND -> +3V3
- J502 pad 15: unconnected-(J502-Pin_15-Pad15) -> Net-(J502-Pin_15)
- J502 pad 17: unconnected-(J502-Pin_17-Pad17) -> Net-(J502-Pin_17)
- J502 pad 19: unconnected-(J502-Pin_19-Pad19) -> Net-(J502-Pin_19)
- J502 pad 2: +3V3 -> GND
- J502 pad 4: unconnected-(J502-Pin_4-Pad4) -> Net-(J502-Pin_4)
- R301 pad 1: ~{User RUN} -> User RUN
- R416 pad 1: Net-(D407-K) -> Net-(D407-A)
- R416 pad 2: GND -> +3V3
- R417 pad 1: Net-(D408-A) -> Net-(D408-K)
- R417 pad 2: +3V3 -> GND
- R419 pad 1: Net-(D410-A) -> Net-(D410-K)
- R419 pad 2: +3V3 -> GND
- R420 pad 1: Net-(D411-K) -> Net-(D411-A)
- R420 pad 2: GND -> +3V3
- R421 pad 1: Net-(D412-A) -> Net-(D412-K)
- R421 pad 2: +3V3 -> GND
- R503 pad 1: +3V3 -> GND
- R503 pad 2: OS Enable Bus 1 -> User Enable Bus 1
- R504 pad 1: +3V3 -> GND
- R504 pad 2: OS Enable Bus 2 -> User Enable Bus 2
- U200 pad 4: ~{User RUN} -> User RUN
- U500 pad 1: OS Enable Bus 1 -> User Enable Bus 1
- U500 pad 28: OS Enable Bus 2 -> User Enable Bus 2
- U500 pad 29: OS Enable Bus 2 -> User Enable Bus 2
- U500 pad 56: OS Enable Bus 1 -> User Enable Bus 1
- U501 pad 14: OS Enable Bus 1 -> User Enable Bus 1
- U501 pad 27: OS Enable Bus 2 -> User Enable Bus 2
- U501 pad 30: GND -> +3V3
- U501 pad 43: GND -> +3V3
Routing:
- net User RUN: track 0.00 -> 128.6 mm, vias 0 -> 5
- net User Enable Bus 1: track 0.00 -> 112.4 mm, vias 0 -> 6
- net User Enable Bus 2: track 0.00 -> 110.9 mm, vias 0 -> 1
- net OS Enable Bus 1: track 104.2 -> 0.00 mm, vias 5 -> 0
- net OS Enable Bus 2: track 104.0 -> 0.00 mm, vias 1 -> 0
- net ~{User RUN}: track 123.0 -> 32.3 mm, vias 3 -> 0
- net Net-(J502-Pin_4): track 0.00 -> 57.6 mm
- net Net-(J502-Pin_15): track 0.00 -> 47.7 mm
- net Net-(J502-Pin_17): track 0.00 -> 45.2 mm
- net Net-(J502-Pin_19): track 0.00 -> 39.1 mm, vias 0 -> 1
- net ~{User Reset}: track 111.5 -> 77.9 mm
- net +3V3: track 316.0 -> 336.1 mm
- net Net-(D410-K): track 0.00 -> 7.76 mm
- net Net-(D412-K): track 0.00 -> 6.71 mm
- net Net-(D412-A): track 6.71 -> 0.00 mm
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Other:
- board text added: "Version 1.1.2"
- board text removed: "Version 1.1"
