File: KiCad/Devkit/Hotswap Pico Hub/debugging.kicad_sch (KiCad schematic)
At the start: 22 parts, among them J1 OS UART, J1 User UART, J401 OS SWD, J405 User SWD, SW403 OS Reset Switch, SW406 User Reset Switch

Commit message: Updated KiCad to V1.1.2
Parts:
- D409: value User Enable Bus 2 -> User Request Bus 1
Connections:
- net OS Enable Bus 1 is gone; now on an unnamed net: D407.2 (A)
- net OS Enable Bus 2 is gone; now on an unnamed net: D411.2 (A)
- net ~{User Enable Bus 1} is gone; now on an unnamed net: D408.1 (K)
- net ~{User Enable Bus 2} is gone; now on an unnamed net: D412.1 (K)
- net ~{User RUN} is gone; now on an unnamed net: D410.1 (K)
- net +3V3: now also R416.2, R420.2; no longer R417.2, R419.2, R421.2
- net GND: now also R417.2, R419.2, R421.2; no longer R416.2, R420.2
- net at R421.1: no longer D412.2 (A)
- net at R417.1: no longer D408.2 (A)
- net at R420.1: no longer D411.1 (K)
- net at R419.1: no longer D410.2 (A)
- net at R416.1: no longer D407.1 (K)
- new net User Enable Bus 1: D408.2 (A)
- new net User Enable Bus 2: D412.2 (A)
- new net User RUN: D410.2 (A)
- new net ~{OS Enable Bus 1}: D407.1 (K)
- new net ~{OS Enable Bus 2}: D411.1 (K)
Other:
- moved on the sheet: D407, D408, D410, D411, D412
