File: KiCad/Devkit/Hotswap Pico Hub/os_pico.kicad_sch (KiCad schematic)
At the start: 3 parts, among them J202 OS SWD In, U1 OS Pico

Commit message: Updated KiCad to V1.1.2
Connections:
- net ~{User RUN} renamed User RUN
Changed lines of the file:
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@@
-    )
-  )
-  (global_label "test" (shape bidirectional) (at 50.8 26.67 180) (fields_autoplaced)
-    (effects (font (size 1.27 1.27)) (justify right))
-    (property "Intersheetrefs" "${INTERSHEET_REFS}" (at 43.1354 26.67 0)
-      (effects (font (size 1.27 1.27)) (justify right) hide)
     )
   )
@@
     )
   )
-  (global_label "~{User RUN}" (shape bidirectional) (at 50.8 39.37 180) (fields_autoplaced)
+  (global_label "User RUN" (shape bidirectional) (at 50.8 39.37 180) (fields_autoplaced)
     (effects (font (size 1.27 1.27)) (justify right))
-    (property "Intersheetrefs" "${INTERSHEET_REFS}" (at 50.8 39.37 0)
-      (effects (font (size 1.27 1.27)) hide)
+    (property "Intersheetrefs" "${INTERSHEET_REFS}" (at 37.5715 39.37 0)
+      (effects (font (size 1.27 1.27)) (justify right) hide)
     )
   )
